File: LogicLevelShifter16/LLS16.brd (EAGLE design)
At the start: 160 x 100 mm, 280 parts, among them J1 0524372471, J2 0524372471, U1 CPH3355-TL-W

Commit message: "Added Capacitors"
Parts:
- added L1-10:C3, L1-10:C4, L1-11:C3, L1-11:C4, L1-12:C3, L1-12:C4, L1-13:C3, L1-13:C4, L1-14:C3, L1-14:C4, L1-15:C3, L1-15:C4, L1-16:C3, L1-16:C4, L1-1:C3, L1-1:C4, L1-2:C3, L1-2:C4, L1-3:C3, L1-3:C4, L1-4:C3, L1-4:C4, L1-5:C3, L1-5:C4, L1-6:C3, L1-6:C4, L1-7:C3, L1-7:C4, L1-8:C3, L1-8:C4, L1-9:C3, L1-9:C4: (no value), rcl:C0805K
- moved L1-10:C1 503.2 mm to (121.9, 243.8)
- moved L1-10:C2 503.2 mm to (121.9, 182.9)
- moved L1-11:C1 503.2 mm to (121.9, 240.0)
- moved L1-15:C2 503.2 mm to (121.9, 163.8)
- moved L1-16:C2 503.2 mm to (121.9, 160.0)
- moved L1-3:C2 503.2 mm to (121.9, 209.6)
- moved L1-4:C2 503.2 mm to (121.9, 205.7)
- moved L1-5:C2 503.2 mm to (121.9, 201.9)
- moved L1-6:C2 503.2 mm to (121.9, 198.1)
- moved L1-7:C2 503.2 mm to (121.9, 194.3)
- moved L1-9:C1 503.2 mm to (121.9, 247.7)
- moved L1-9:C2 503.2 mm to (121.9, 186.7)
- moved L1-11:C2 503.2 mm to (121.9, 179.1)
- moved L1-12:C1 503.2 mm to (121.9, 236.2)
- moved L1-12:C2 503.2 mm to (121.9, 175.3)
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Connections:
- net +3V: now also L1-10:C3.1, L1-10:C4.1, L1-11:C3.1, L1-11:C4.1, L1-12:C3.1, L1-12:C4.1, L1-13:C3.1, L1-13:C4.1, L1-14:C3.1, L1-14:C4.1, L1-15:C3.1, L1-15:C4.1, L1-16:C3.1, L1-16:C4.1, L1-1:C3.1, L1-1:C4.1, L1-2:C3.1, L1-2:C4.1, L1-3:C3.1, L1-3:C4.1, L1-4:C3.1, L1-4:C4.1, L1-5:C3.1, L1-5:C4.1, L1-6:C3.1, L1-6:C4.1, L1-7:C3.1, L1-7:C4.1, L1-8:C3.1, L1-8:C4.1, L1-9:C3.1, L1-9:C4.1
- net GND: now also L1-10:C3.2, L1-10:C4.2, L1-11:C3.2, L1-11:C4.2, L1-12:C3.2, L1-12:C4.2, L1-13:C3.2, L1-13:C4.2, L1-14:C3.2, L1-14:C4.2, L1-15:C3.2, L1-15:C4.2, L1-16:C3.2, L1-16:C4.2, L1-1:C3.2, L1-1:C4.2, L1-2:C3.2, L1-2:C4.2, L1-3:C3.2, L1-3:C4.2, L1-4:C3.2, L1-4:C4.2, L1-5:C3.2, L1-5:C4.2, L1-6:C3.2, L1-6:C4.2, L1-7:C3.2, L1-7:C4.2, L1-8:C3.2, L1-8:C4.2, L1-9:C3.2, L1-9:C4.2
Routing:
- net -1.5V: track 0.00 -> 1662.0 mm, vias 0 -> 34
- net F1: track 0.00 -> 1093.7 mm
- net F15: track 0.00 -> 1063.1 mm
- net +3V: track 0.00 -> 924.5 mm, vias 0 -> 24
- net M16: track 0.00 -> 799.8 mm
- net M14: track 0.00 -> 770.5 mm
- net M15: track 0.00 -> 741.9 mm
- net M1: track 0.00 -> 735.6 mm
- net L1-9:N$10: track 0.00 -> 439.3 mm
- net L1-4:N$10: track 0.00 -> 418.3 mm
- net L1-9:N$3: track 0.00 -> 372.9 mm
- net L1-4:N$3: track 0.00 -> 369.2 mm
- net L1-6:N$3: track 0.00 -> 363.9 mm
- net GND: track 0.00 -> 344.8 mm, vias 0 -> 7
- net L1-1:N$8: track 0.00 -> 329.2 mm
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Other:
- board size 160 x 100 mm -> 346.7 x 491.2 mm
